Commit message: Convert visual meshes to obj (#203)
Co-authored-by: David von Wrangel <wrangelvid@gmail.como>

File: spot_description/urdf/accessories.urdf.xacro (robot description, xacro)
@@ -10,15 +10,15 @@
       <visual>
         <geometry>
-          <mesh filename="package://spot_description/meshes/base/visual/pack_top.dae"/>
+          <mesh filename="package://spot_description/meshes/base/visual/pack_top.obj"/>
         </geometry>
       </visual>
       <visual>
         <geometry>
-          <mesh filename="package://spot_description/meshes/base/visual/pack_body.dae"/>
+          <mesh filename="package://spot_description/meshes/base/visual/pack_body.obj"/>
         </geometry>
       </visual>
       <collision>
         <geometry>
-          <mesh filename="package://spot_description/meshes/base/visual/pack_body.dae"/>
+          <mesh filename="package://spot_description/meshes/base/visual/pack_body.obj"/>
         </geometry>
       </collision>
@@ -34,5 +34,5 @@
       <visual>
         <geometry>
-          <mesh filename="package://spot_description/meshes/base/visual/lidar_mount.dae"/>
+          <mesh filename="package://spot_description/meshes/base/visual/lidar_mount.obj"/>
         </geometry>
       </visual>

File: spot_description/urdf/spot_macro.xacro (robot description, xacro)
@@ -7,5 +7,5 @@
             <visual>
                 <geometry>
-                    <mesh filename="package://spot_description/meshes/base/visual/body.dae" />
+                    <mesh filename="package://spot_description/meshes/base/visual/body.obj" />
                 </geometry>
             </visual>
@@ -59,5 +59,5 @@
                 <geometry>
                     <mesh
-                        filename="package://spot_description/meshes/base/visual/front_left_hip.dae" />
+                        filename="package://spot_description/meshes/base/visual/front_left_hip.obj" />
                 </geometry>
             </visual>
@@ -82,5 +82,5 @@
                 <geometry>
                     <mesh
-                        filename="package://spot_description/meshes/base/visual/front_left_upper_leg.dae" />
+                        filename="package://spot_description/meshes/base/visual/front_left_upper_leg.obj" />
                 </geometry>
             </visual>
@@ -111,5 +111,5 @@
                 <geometry>
                     <mesh
-                        filename="package://spot_description/meshes/base/visual/front_left_lower_leg.dae" />
+                        filename="package://spot_description/meshes/base/visual/front_left_lower_leg.obj" />
                 </geometry>
             </visual>
@@ -145,5 +145,5 @@
                 <geometry>
                     <mesh
-                        filename="package://spot_description/meshes/base/visual/front_right_hip.dae" />
+                        filename="package://spot_description/meshes/base/visual/front_right_hip.obj" />
                 </geometry>
             </visual>
@@ -168,5 +168,5 @@
                 <geometry>
                     <mesh
-                        filename="package://spot_description/meshes/base/visual/front_right_upper_leg.dae" />
+                        filename="package://spot_description/meshes/base/visual/front_right_upper_leg.obj" />
                 </geometry>
             </visual>
@@ -197,5 +197,5 @@
                 <geometry>
                     <mesh
-                        filename="package://spot_description/meshes/base/visual/front_right_lower_leg.dae" />
+                        filename="package://spot_description/meshes/base/visual/front_right_lower_leg.obj" />
                 </geometry>
             </visual>
@@ -231,5 +231,5 @@
                 <geometry>
                     <mesh
-                        filename="package://spot_description/meshes/base/visual/rear_left_hip.dae" />
+                        filename="package://spot_description/meshes/base/visual/rear_left_hip.obj" />
                 </geometry>
             </visual>
@@ -254,5 +254,5 @@
                 <geometry>
                     <mesh
-                        filename="package://spot_description/meshes/base/visual/rear_left_upper_leg.dae" />
+                        filename="package://spot_description/meshes/base/visual/rear_left_upper_leg.obj" />
                 </geometry>
             </visual>
@@ -283,5 +283,5 @@
                 <geometry>
                     <mesh
-                        filename="package://spot_description/meshes/base/visual/rear_left_lower_leg.dae" />
+                        filename="package://spot_description/meshes/base/visual/rear_left_lower_leg.obj" />
                 </geometry>
             </visual>
@@ -317,5 +317,5 @@
                 <geometry>
                     <mesh
-                        filename="package://spot_description/meshes/base/visual/rear_right_hip.dae" />
+                        filename="package://spot_description/meshes/base/visual/rear_right_hip.obj" />
                 </geometry>
             </visual>
@@ -340,5 +340,5 @@
                 <geometry>
                     <mesh
-                        filename="package://spot_description/meshes/base/visual/rear_right_upper_leg.dae" />
+                        filename="package://spot_description/meshes/base/visual/rear_right_upper_leg.obj" />
                 </geometry>
             </visual>
@@ -369,5 +369,5 @@
                 <geometry>
                     <mesh
-                        filename="package://spot_description/meshes/base/visual/rear_right_lower_leg.dae" />
+                        filename="package://spot_description/meshes/base/visual/rear_right_lower_leg.obj" />
                 </geometry>
             </visual>
