Commit message: [N/A] Convexified collision geometries (#164)
Co-authored-by: David von Wrangel <wrangelvid@gmail.como>

File: spot_description/urdf/spot_macro.xacro (robot description, xacro)
@@ -13,5 +13,5 @@
                 <geometry>
                     <mesh
-                        filename="file://$(find spot_description)/meshes/base/collision/body_collision.stl" />
+                        filename="file://$(find spot_description)/meshes/base/collision/body_collision.obj" />
                 </geometry>
             </collision>
@@ -62,10 +62,4 @@
                 </geometry>
             </visual>
-            <collision>
-                <geometry>
-                    <mesh
-                        filename="file://$(find spot_description)/meshes/base/collision/front_left_hip_collision.stl" />
-                </geometry>
-            </collision>
             <inertial>
                 <origin rpy="-0.716521349312305 0.02956473059648479 0.03655230014702582"
@@ -94,5 +88,5 @@
                 <geometry>
                     <mesh
-                        filename="file://$(find spot_description)/meshes/base/collision/front_left_upper_leg_collision.stl" />
+                        filename="file://$(find spot_description)/meshes/base/collision/left_upper_leg_collision.obj" />
                 </geometry>
             </collision>
@@ -123,5 +117,11 @@
                 <geometry>
                     <mesh
-                        filename="file://$(find spot_description)/meshes/base/collision/front_left_lower_leg_collision.stl" />
+                        filename="file://$(find spot_description)/meshes/base/collision/left_lower_leg_collision.obj" />
+                </geometry>
+            </collision>
+            <collision>
+                <origin xyz="0.0 0.0 -0.3365" rpy="0 0 0" />
+                <geometry>
+                    <sphere radius="0.036"/>
                 </geometry>
             </collision>
@@ -148,10 +148,4 @@
                 </geometry>
             </visual>
-            <collision>
-                <geometry>
-                    <mesh
-                        filename="file://$(find spot_description)/meshes/base/collision/front_right_hip_collision.stl" />
-                </geometry>
-            </collision>
             <inertial>
                 <origin rpy="0.7165213493123055 -0.02956473059648479 0.03655230014702582"
@@ -180,5 +174,5 @@
                 <geometry>
                     <mesh
-                        filename="file://$(find spot_description)/meshes/base/collision/front_right_upper_leg_collision.stl" />
+                        filename="file://$(find spot_description)/meshes/base/collision/right_upper_leg_collision.obj" />
                 </geometry>
             </collision>
@@ -209,5 +203,11 @@
                 <geometry>
                     <mesh
-                        filename="file://$(find spot_description)/meshes/base/collision/front_right_lower_leg_collision.stl" />
+                        filename="file://$(find spot_description)/meshes/base/collision/right_lower_leg_collision.obj" />
+                </geometry>
+            </collision>
+            <collision>
+                <origin xyz="0.0 0.0 -0.3365" rpy="0 0 0" />
+                <geometry>
+                    <sphere radius="0.036"/>
                 </geometry>
             </collision>
@@ -234,10 +234,4 @@
                 </geometry>
             </visual>
-            <collision>
-                <geometry>
-                    <mesh
-                        filename="file://$(find spot_description)/meshes/base/collision/rear_left_hip_collision.stl" />
-                </geometry>
-            </collision>
             <inertial>
                 <origin rpy="0.7165213493123055 -0.02956473059648479 0.03655230014702582"
@@ -266,5 +260,5 @@
                 <geometry>
                     <mesh
-                        filename="file://$(find spot_description)/meshes/base/collision/rear_left_upper_leg_collision.stl" />
+                        filename="file://$(find spot_description)/meshes/base/collision/left_upper_leg_collision.obj" />
                 </geometry>
             </collision>
@@ -295,5 +289,11 @@
                 <geometry>
                     <mesh
-                        filename="file://$(find spot_description)/meshes/base/collision/rear_left_lower_leg_collision.stl" />
+                        filename="file://$(find spot_description)/meshes/base/collision/left_lower_leg_collision.obj" />
+                </geometry>
+            </collision>
+            <collision>
+                <origin xyz="0.0 0.0 -0.3365" rpy="0 0 0" />
+                <geometry>
+                    <sphere radius="0.036"/>
                 </geometry>
             </collision>
@@ -320,10 +320,4 @@
                 </geometry>
             </visual>
-            <collision>
-                <geometry>
-                    <mesh
-                        filename="file://$(find spot_description)/meshes/base/collision/rear_right_hip_collision.stl" />
-                </geometry>
-            </collision>
             <inertial>
                 <origin rpy="0.7165213493123055 -0.02956473059648479 0.03655230014702582"
@@ -352,5 +346,5 @@
                 <geometry>
                     <mesh
-                        filename="file://$(find spot_description)/meshes/base/collision/rear_right_upper_leg_collision.stl" />
+                        filename="file://$(find spot_description)/meshes/base/collision/right_upper_leg_collision.obj" />
                 </geometry>
             </collision>
@@ -381,5 +375,11 @@
                 <geometry>
                     <mesh
-                        filename="file://$(find spot_description)/meshes/base/collision/rear_right_lower_leg_collision.stl" />
+                        filename="file://$(find spot_description)/meshes/base/collision/right_lower_leg_collision.obj" />
+                </geometry>
+            </collision>
+            <collision>
+                <origin xyz="0.0 0.0 -0.3365" rpy="0 0 0" />
+                <geometry>
+                    <sphere radius="0.036"/>
                 </geometry>
             </collision>

Commit message: Update joint effort values in URDF (#429)

File: spot_description/urdf/spot_macro.xacro (robot description, xacro)
@@ -75,5 +75,5 @@
             <parent link="${tf_prefix}body" />
             <child link="${tf_prefix}front_left_hip" />
-            <limit effort="1000" velocity="1000.00" lower="-0.78539816339744827899"
+            <limit effort="45" velocity="1000.00" lower="-0.78539816339744827899"
                 upper="0.78539816339744827899" />
         </joint>
@@ -104,5 +104,5 @@
             <parent link="${tf_prefix}front_left_hip" />
             <child link="${tf_prefix}front_left_upper_leg" />
-            <limit effort="1000" velocity="1000.00" lower="-0.89884456477707963539"
+            <limit effort="45" velocity="1000.00" lower="-0.89884456477707963539"
                 upper="2.2951079663725435509" />
         </joint>
@@ -139,5 +139,5 @@
             <parent link="${tf_prefix}front_left_upper_leg" />
             <child link="${tf_prefix}front_left_lower_leg" />
-            <limit effort="1000" velocity="1000.00" lower="-2.7929" upper="-0.254801" />
+            <limit effort="115" velocity="1000.00" lower="-2.7929" upper="-0.254801" />
         </joint>
         <link name="${tf_prefix}front_right_hip">
@@ -161,5 +161,5 @@
             <parent link="${tf_prefix}body" />
             <child link="${tf_prefix}front_right_hip" />
-            <limit effort="1000" velocity="1000.00" lower="-0.78539816339744827899"
+            <limit effort="45" velocity="1000.00" lower="-0.78539816339744827899"
                 upper="0.78539816339744827899" />
         </joint>
@@ -190,5 +190,5 @@
             <parent link="${tf_prefix}front_right_hip" />
             <child link="${tf_prefix}front_right_upper_leg" />
-            <limit effort="1000" velocity="1000.00" lower="-0.89884456477707963539"
+            <limit effort="45" velocity="1000.00" lower="-0.89884456477707963539"
                 upper="2.2951079663725435509" />
         </joint>
@@ -225,5 +225,5 @@
             <parent link="${tf_prefix}front_right_upper_leg" />
             <child link="${tf_prefix}front_right_lower_leg" />
-            <limit effort="1000" velocity="1000.00" lower="-2.7929" upper="-0.247563" />
+            <limit effort="115" velocity="1000.00" lower="-2.7929" upper="-0.247563" />
         </joint>
         <link name="${tf_prefix}rear_left_hip">
@@ -247,5 +247,5 @@
             <parent link="${tf_prefix}body" />
             <child link="${tf_prefix}rear_left_hip" />
-            <limit effort="1000" velocity="1000.00" lower="-0.78539816339744827899"
+            <limit effort="45" velocity="1000.00" lower="-0.78539816339744827899"
                 upper="0.78539816339744827899" />
         </joint>
@@ -276,5 +276,5 @@
             <parent link="${tf_prefix}rear_left_hip" />
             <child link="${tf_prefix}rear_left_upper_leg" />
-            <limit effort="1000" velocity="1000.00" lower="-0.89884456477707963539"
+            <limit effort="45" velocity="1000.00" lower="-0.89884456477707963539"
                 upper="2.2951079663725435509" />
         </joint>
@@ -311,5 +311,5 @@
             <parent link="${tf_prefix}rear_left_upper_leg" />
             <child link="${tf_prefix}rear_left_lower_leg" />
-            <limit effort="1000" velocity="1000.00" lower="-2.7929" upper="-0.267153" />
+            <limit effort="115" velocity="1000.00" lower="-2.7929" upper="-0.267153" />
         </joint>
         <link name="${tf_prefix}rear_right_hip">
@@ -333,5 +333,5 @@
             <parent link="${tf_prefix}body" />
             <child link="${tf_prefix}rear_right_hip" />
-            <limit effort="1000" velocity="1000.00" lower="-0.78539816339744827899"
+            <limit effort="45" velocity="1000.00" lower="-0.78539816339744827899"
                 upper="0.78539816339744827899" />
         </joint>
@@ -362,5 +362,5 @@
             <parent link="${tf_prefix}rear_right_hip" />
             <child link="${tf_prefix}rear_right_upper_leg" />
-            <limit effort="1000" velocity="1000.00" lower="-0.89884456477707963539"
+            <limit effort="45" velocity="1000.00" lower="-0.89884456477707963539"
                 upper="2.2951079663725435509" />
         </joint>
@@ -397,5 +397,5 @@
             <parent link="${tf_prefix}rear_right_upper_leg" />
             <child link="${tf_prefix}rear_right_lower_leg" />
-            <limit effort="1000" velocity="1000.00" lower="-2.7929" upper="-0.257725" />
+            <limit effort="115" velocity="1000.00" lower="-2.7929" upper="-0.257725" />
         </joint>
         <!-- Standard accessories. -->
